File: hardware/rev2/expansion.kicad_sch (KiCad schematic)
At the start: 1 part, among them J7 Expansion Header

Commit message: fix(hardware): assign missing footprints to J6, J7, JP1, JP2
The four remaining symbols without footprints blocked Update PCB from
Schematic. J6/J7 get vertical 2.54 mm pin headers; JP1/JP2 get the
open TrianglePad solder jumper, matching the design default of an open
MODE jumper (floating = active-HIGH) and easy to bridge with an iron.

All 172 symbol instances across the eight sheets now carry a footprint.

Co-Authored-By: Claude Fable 5 <noreply@anthropic.com>
Parts:
- J7: footprint (none) -> Connector_PinHeader_2.54mm:PinHeader_1x08_P2.54mm_Vertical
Changed lines of the file:
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@@
 			)
 		)
-		(property "Footprint" ""
+		(property "Footprint" "Connector_PinHeader_2.54mm:PinHeader_1x08_P2.54mm_Vertical"
 			(at 110.49 74.93 0)
 			(hide yes)
