File: hardware/rev2/level-sensors.kicad_sch (KiCad schematic)
At the start: 12 parts, among them J10 RESERVOIR_HIGH, J5 RESERVOIR_LOW, Q1 2N7002, Q81 2N7002

Commit message: fix(hardware): assign missing footprints to J6, J7, JP1, JP2
The four remaining symbols without footprints blocked Update PCB from
Schematic. J6/J7 get vertical 2.54 mm pin headers; JP1/JP2 get the
open TrianglePad solder jumper, matching the design default of an open
MODE jumper (floating = active-HIGH) and easy to bridge with an iron.

All 172 symbol instances across the eight sheets now carry a footprint.

Co-Authored-By: Claude Fable 5 <noreply@anthropic.com>
Parts:
- JP1, JP2: footprint (none) -> Jumper:SolderJumper-2_P1.3mm_Open_TrianglePad1.0x1.5mm
Changed lines of the file:
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@@
 			)
 		)
-		(property "Footprint" ""
+		(property "Footprint" "Jumper:SolderJumper-2_P1.3mm_Open_TrianglePad1.0x1.5mm"
 			(at 60.96 104.14 0)
 			(hide yes)
@@
 			)
 		)
-		(property "Footprint" ""
+		(property "Footprint" "Jumper:SolderJumper-2_P1.3mm_Open_TrianglePad1.0x1.5mm"
 			(at 179.07 104.14 0)
 			(hide yes)
